File: PCB/DYI_CDJ_v1/DYI_CDJ_v1.kicad_pcb (KiCad board)
At the start: 2 copper layers, 240 x 135 mm, 55 parts, among them SW1 SW_Push, SW10 SW_Push, SW11 SW_Push, SW12 SW_Push, SW13 SW_Push, SW14 SW_Push, SW15 SW_Push, SW16 SW_Push, SW17 RotaryEncoder, SW18 RotaryEncoder, SW19 SW_Push, SW2 SW_Push, SW20 SW_Push, SW21 RotaryEncoder, SW3 SW_Push, SW4 SW_Push, SW5 SW_Push, SW6 SW_Push, SW7 SW_Push, SW8 SW_Push, SW9 SW_Push, U1 Arduino_Pro_Micro_USB_C, U2 CD74HC4067_Module_Generic, U3 PCF8575_Module_HW331

Commit message: PCB update dev
Parts:
- R1, R10, R11, R12, R13, R14, R15, R16, R2, R3, R4, R5, R6, R7, R8, R9: footprint Resistor_SMD:R_0603_1608Metric -> Resistor_THT:R_Axial_DIN0207_L6.3mm_D2.5mm_P10.16mm_Horizontal
- moved SW20 170.3 mm to (46.0, 129.5)
- moved SW9 162.9 mm to (231.0, 104.5)
- moved SW14 160.7 mm to (162.2, 36.5)
- moved SW15 150.5 mm to (236.5, 147.5)
- moved SW16 150.5 mm to (236.5, 129.5)
- moved SW4 146.7 mm to (51.5, 104.5)
- moved SW6 144.3 mm to (69.5, 142.5)
- moved SW10 133.9 mm to (68.0, 104.5)
- moved SW12 127.0 mm to (86.0, 142.5)
- moved SW13 119.0 mm to (120.2, 36.5)
- moved SW1 118.3 mm to (196.4, 127.0)
- moved SW7 103.8 mm to (213.0, 127.0)
- moved R1 65.7 mm to (184.0, 77.0), turned to 0 degrees
- moved R2 65.7 mm to (184.0, 74.5), turned to 0 degrees
- moved R4 64.8 mm to (184.0, 92.3), turned to 0 degrees
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- renumbered SW13 to SW1, SW2 to SW10, SW6 to SW11, SW8 to SW12, SW19 to SW13, SW20 to SW14, SW12 to SW15, SW11 to SW16, SW4 to SW19, SW15 to SW2, SW3 to SW20, SW9 to SW3, SW1 to SW4, SW7 to SW6, SW14 to SW7, SW16 to SW8, SW10 to SW9
Connections:
- U3 pad P00: /But_loopIn_D1 -> /But_loopOut_D1
- U3 pad P01: /But_loopOut_D1 -> /But_loopIn_D1
- U3 pad P02: /But_Cue_D1 -> /But_Pad3_D1
- U3 pad P03: /But_Play_D1 -> /But_Pad4_D1
- U3 pad P06: /But_Pad3_D1 -> /But_Cue_D1
- U3 pad P07: /But_Pad4_D1 -> /But_Play_D1
- U3 pad P10: /But_loopIn_D2 -> /But_Pad4_D2
- U3 pad P11: /But_loopOut_D2 -> /But_Pad3_D2
- U3 pad P12: /But_Cue_D2 -> /But_Pad1_D2
- U3 pad P13: /But_Play_D2 -> /But_Pad2_D2
- U3 pad P14: /But_Pad1_D2 -> /But_Cue_D2
- U3 pad P15: /But_Pad2_D2 -> /But_Play_D2
- U3 pad P16: /But_Pad3_D2 -> /But_loopIn_D2
- U3 pad P17: /But_Pad4_D2 -> /But_loopOut_D2
Routing:
- net GND: track 0.00 -> 1254.4 mm
- net +5V: track 0.00 -> 636.3 mm, vias 0 -> 2
- net /But_loopIn_D1: track 0.00 -> 202.7 mm, vias 0 -> 2
- net /But_Play_D1: track 0.00 -> 186.4 mm, vias 0 -> 2
- net /JoggingPinA_D2: track 0.00 -> 183.2 mm
- net /But_Pad3_D1: track 0.00 -> 179.5 mm, vias 0 -> 1
- net /But_Pad2_D1: track 0.00 -> 177.9 mm, vias 0 -> 1
- net /But_loopOut_D1: track 0.00 -> 177.0 mm
- net /JoggingPinB_D2: track 0.00 -> 174.6 mm
- net /But_Cue_D1: track 0.00 -> 174.3 mm, vias 0 -> 1
- net /But_Pad4_D1: track 0.00 -> 167.2 mm, vias 0 -> 2
- net /But_Pad1_D1: track 0.00 -> 164.1 mm, vias 0 -> 1
- net /But_Pad2_D2: track 4.57 -> 152.4 mm
- net /i2c_SDA: track 0.00 -> 147.7 mm
- net /i2c_SCL: track 0.00 -> 144.0 mm
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Other:
- board text removed: "${REFERENCE}"
