File: PCB/DYI_CDJ_v1/DYI_CDJ_v1.kicad_sch (KiCad schematic)
At the start: 55 parts, among them SW1 SW_Push, SW10 SW_Push, SW11 SW_Push, SW12 SW_Push, SW13 SW_Push, SW14 SW_Push, SW15 SW_Push, SW16 SW_Push, SW17 RotaryEncoder, SW18 RotaryEncoder, SW19 SW_Push, SW2 SW_Push, SW20 SW_Push, SW21 RotaryEncoder, SW3 SW_Push, SW4 SW_Push, SW5 SW_Push, SW6 SW_Push, SW7 SW_Push, SW8 SW_Push, SW9 SW_Push, U1 Arduino_Pro_Micro_USB_C, U2 CD74HC4067_Module_Generic, U3 PCF8575_Module_HW331

Commit message: PCB update dev
Parts:
- R1, R10, R11, R12, R13, R14, R15, R16, R2, R3, R4, R5, R6, R7, R8, R9: footprint Resistor_SMD:R_0603_1608Metric -> Resistor_THT:R_Axial_DIN0207_L6.3mm_D2.5mm_P10.16mm_Horizontal
- renumbered SW13 to SW1, SW2 to SW10, SW6 to SW11, SW8 to SW12, SW19 to SW13, SW20 to SW14, SW12 to SW15, SW11 to SW16, SW4 to SW19, SW15 to SW2, SW3 to SW20, SW9 to SW3, SW1 to SW4, SW7 to SW6, SW14 to SW7, SW16 to SW8, SW10 to SW9
Connections:
- net But_Cue_D1: now also U3.P06; no longer U3.P02
- net But_Cue_D2: now also U3.P14; no longer U3.P12
- net But_Pad1_D2: now also U3.P12; no longer U3.P14
- net But_Pad2_D2: now also U3.P13; no longer U3.P15
- net But_Pad3_D1: now also U3.P02; no longer U3.P06
- net But_Pad3_D2: now also U3.P11; no longer U3.P16
- net But_Pad4_D1: now also U3.P03; no longer U3.P07
- net But_Pad4_D2: now also U3.P10; no longer U3.P17
- net But_Play_D1: now also U3.P07; no longer U3.P03
- net But_Play_D2: now also U3.P15; no longer U3.P13
- net But_loopIn_D1: now also U3.P01; no longer U3.P00
- net But_loopIn_D2: now also U3.P16; no longer U3.P10
- net But_loopOut_D1: now also U3.P00; no longer U3.P01
- net But_loopOut_D2: now also U3.P17; no longer U3.P11
Changed lines of the file:
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@@
 		)
 	)
-	(label "But_Pad3_D2"
+	(label "But_loopIn_D2"
 		(at 234.95 107.95 0)
 		(effects
@@
 		)
 	)
-	(label "But_loopOut_D1"
+	(label "But_loopIn_D1"
 		(at 234.95 74.93 0)
 		(effects
@@
 		)
 	)
-	(label "But_Play_D1"
+	(label "But_Pad4_D1"
 		(at 234.95 80.01 0)
 		(effects
@@
 		)
 	)
-	(label "But_Pad4_D2"
+	(label "But_loopOut_D2"
 		(at 234.95 110.49 0)
 		(effects
@@
 		)
 	)
-	(label "But_Pad2_D2"
+	(label "But_Play_D2"
 		(at 234.95 105.41 0)
 		(effects
@@
 		)
 	)
-	(label "But_Cue_D2"
+	(label "But_Pad1_D2"
 		(at 234.95 97.79 0)
 		(effects
@@
 		)
 	)
-	(label "But_loopIn_D1"
+	(label "But_loopOut_D1"
 		(at 234.95 72.39 0)
 		(effects
@@
 		)
 	)
-	(label "But_Pad3_D1"
+	(label "But_Cue_D1"
 		(at 234.95 87.63 0)
 		(effects
@@
 		)
 	)
-	(label "But_loopIn_D2"
+	(label "But_Pad4_D2"
 		(at 234.95 92.71 0)
 		(effects
@@
 		)
 	)
-	(label "But_loopOut_D2"
+	(label "But_Pad3_D2"
 		(at 234.95 95.25 0)
 		(effects
@@
 		)
 	)
-	(label "But_Play_D2"
+	(label "But_Pad2_D2"
 		(at 234.95 100.33 0)
 		(effects
@@
 		)
 	)
-	(label "But_Pad1_D2"
+	(label "But_Cue_D2"
 		(at 234.95 102.87 0)
 		(effects
@@
 		)
 	)
-	(label "But_Pad4_D1"
+	(label "But_Play_D1"
 		(at 234.95 90.17 0)
 		(effects
@@
 		)
 	)
-	(label "But_Cue_D1"
+	(label "But_Pad3_D1"
 		(at 234.95 77.47 0)
 		(effects
@@
 			)
 		)
-		(property "Footprint" "Resistor_SMD:R_0603_1608Metric"
+		(property "Footprint" "Resistor_THT:R_Axial_DIN0207_L6.3mm_D2.5mm_P10.16mm_Horizontal"
 			(at 35.56 220.218 90)
 			(effects
@@
 		(dnp no)
 		(fields_autoplaced yes)
-		(property "Reference" "SW14"
+		(property "Reference" "SW7"
 			(at 62.23 237.49 0)
 			(effects
@@
 			(project "DYI_CDJ_v1"
 				(path "/f67f3c27-8ae6-4ed2-82a6-2d91869979e0"
-					(reference "SW14")
+					(reference "SW7")
 					(unit 1)
 				)
@@
 		(dnp no)
 		(fields_autoplaced yes)
-		(property "Reference" "SW19"
+		(property "Reference" "SW13"
 			(at 137.16 33.02 0)
 			(effects
@@
 			(project "DYI_CDJ_v1"
 				(path "/f67f3c27-8ae6-4ed2-82a6-2d91869979e0"
-					(reference "SW19")
+					(reference "SW13")
 					(unit 1)
 				)
@@
 		(dnp no)
 		(fields_autoplaced yes)
-		(property "Reference" "SW6"
+		(property "Reference" "SW11"
 			(at 62.23 114.3 0)
 			(effects
@@
 			(project "DYI_CDJ_v1"
 				(path "/f67f3c27-8ae6-4ed2-82a6-2d91869979e0"
-					(reference "SW6")
+					(reference "SW11")
 					(unit 1)
 				)
@@
 		(dnp no)
 		(fields_autoplaced yes)
-		(property "Reference" "SW7"
+		(property "Reference" "SW6"
 			(at 62.23 132.08 0)
 			(effects
@@
 			(project "DYI_CDJ_v1"
 				(path "/f67f3c27-8ae6-4ed2-82a6-2d91869979e0"
-					(reference "SW7")
+					(reference "SW6")
 					(unit 1)
 				)
@@
 		(dnp no)
 		(fields_autoplaced yes)
-		(property "Reference" "SW9"
+		(property "Reference" "SW3"
 			(at 62.23 162.56 0)
 			(effects
@@
 			(project "DYI_CDJ_v1"
 				(path "/f67f3c27-8ae6-4ed2-82a6-2d91869979e0"
-					(reference "SW9")
+					(reference "SW3")
 					(unit 1)
 				)
@@
 			)
 		)
-		(property "Footprint" "Resistor_SMD:R_0603_1608Metric"
+		(property "Footprint" "Resistor_THT:R_Axial_DIN0207_L6.3mm_D2.5mm_P10.16mm_Horizontal"
 			(at 35.56 141.478 90)
 			(effects
@@
 		(dnp no)
 		(fields_autoplaced yes)
-		(property "Reference" "SW13"
+		(property "Reference" "SW1"
 			(at 62.23 224.79 0)
 			(effects
@@
 			(project "DYI_CDJ_v1"
 				(path "/f67f3c27-8ae6-4ed2-82a6-2d91869979e0"
-					(reference "SW13")
+					(reference "SW1")
 					(unit 1)
 				)
@@
 		(dnp no)
 		(fields_autoplaced yes)
-		(property "Reference" "SW10"
+		(property "Reference" "SW9"
 			(at 62.23 177.8 0)
 			(effects
@@
 			(project "DYI_CDJ_v1"
 				(path "/f67f3c27-8ae6-4ed2-82a6-2d91869979e0"
-					(reference "SW10")
+					(reference "SW9")
 					(unit 1)
 				)
@@
 			)
 		)
-		(property "Footprint" "Resistor_SMD:R_0603_1608Metric"
+		(property "Footprint" "Resistor_THT:R_Axial_DIN0207_L6.3mm_D2.5mm_P10.16mm_Horizontal"
 			(at 35.56 246.888 90)
 			(effects
@@
 			)
 		)
-		(property "Footprint" "Resistor_SMD:R_0603_1608Metric"
+		(property "Footprint" "Resistor_THT:R_Axial_DIN0207_L6.3mm_D2.5mm_P10.16mm_Horizontal"
 			(at 35.56 104.648 90)
 			(effects
@@
 		(dnp no)
 		(fields_autoplaced yes)
-		(property "Reference" "SW16"
+		(property "Reference" "SW8"
 			(at 62.23 270.51 0)
 			(effects
@@
 			(project "DYI_CDJ_v1"
 				(path "/f67f3c27-8ae6-4ed2-82a6-2d91869979e0"
-					(reference "SW16")
+					(reference "SW8")
 					(unit 1)
 				)
@@
 			)
 		)
-		(property "Footprint" "Resistor_SMD:R_0603_1608Metric"
+		(property "Footprint" "Resistor_THT:R_Axial_DIN0207_L6.3mm_D2.5mm_P10.16mm_Horizontal"
 			(at 35.56 171.958 90)
 			(effects
@@
 		(dnp no)
 		(fields_autoplaced yes)
-		(property "Reference" "SW1"
+		(property "Reference" "SW4"
 			(at 62.23 22.86 0)
 			(effects
@@
 			(project ""
 				(path "/f67f3c27-8ae6-4ed2-82a6-2d91869979e0"
-					(reference "SW1")
+					(reference "SW4")
 					(unit 1)
 				)
@@
 			)
 		)
-		(property "Footprint" "Resistor_SMD:R_0603_1608Metric"
+		(property "Footprint" "Resistor_THT:R_Axial_DIN0207_L6.3mm_D2.5mm_P10.16mm_Horizontal"
 			(at 35.56 70.358 90)
 			(effects
@@
 			)
 		)
-		(property "Footprint" "Resistor_SMD:R_0603_1608Metric"
+		(property "Footprint" "Resistor_THT:R_Axial_DIN0207_L6.3mm_D2.5mm_P10.16mm_Horizontal"
 			(at 35.56 156.718 90)
 			(effects
@@
 		(dnp no)
 		(fields_autoplaced yes)
-		(property "Reference" "SW4"
+		(property "Reference" "SW19"
 			(at 62.23 78.74 0)
 			(effects
@@
 			(project "DYI_CDJ_v1"
 				(path "/f67f3c27-8ae6-4ed2-82a6-2d91869979e0"
-					(reference "SW4")
+					(reference "SW19")
 					(unit 1)
 				)
@@
 		(dnp no)
 		(fields_autoplaced yes)
-		(property "Reference" "SW20"
+		(property "Reference" "SW14"
 			(at 137.16 45.72 0)
 			(effects
@@
 			(project "DYI_CDJ_v1"
 				(path "/f67f3c27-8ae6-4ed2-82a6-2d91869979e0"
-					(reference "SW20")
+					(reference "SW14")
 					(unit 1)
 				)
@@
 		(dnp no)
 		(fields_autoplaced yes)
-		(property "Reference" "SW11"
+		(property "Reference" "SW16"
 			(at 62.23 195.58 0)
 			(effects
@@
 			(project "DYI_CDJ_v1"
 				(path "/f67f3c27-8ae6-4ed2-82a6-2d91869979e0"
-					(reference "SW11")
+					(reference "SW16")
 					(unit 1)
 				)
@@
 			)
 		)
-		(property "Footprint" "Resistor_SMD:R_0603_1608Metric"
+		(property "Footprint" "Resistor_THT:R_Axial_DIN0207_L6.3mm_D2.5mm_P10.16mm_Horizontal"
 			(at 35.56 88.138 90)
 			(effects
@@
 		(dnp no)
 		(fields_autoplaced yes)
-		(property "Reference" "SW2"
+		(property "Reference" "SW10"
 			(at 62.23 41.91 0)
 			(effects
@@
 			(project "DYI_CDJ_v1"
 				(path "/f67f3c27-8ae6-4ed2-82a6-2d91869979e0"
-					(reference "SW2")
+					(reference "SW10")
 					(unit 1)
 				)
@@
 		(dnp no)
 		(fields_autoplaced yes)
-		(property "Reference" "SW8"
+		(property "Reference" "SW12"
 			(at 62.23 147.32 0)
 			(effects
@@
 			(project "DYI_CDJ_v1"
 				(path "/f67f3c27-8ae6-4ed2-82a6-2d91869979e0"
-					(reference "SW8")
+					(reference "SW12")
 					(unit 1)
 				)
@@
 			)
 		)
-		(property "Footprint" "Resistor_SMD:R_0603_1608Metric"
+		(property "Footprint" "Resistor_THT:R_Axial_DIN0207_L6.3mm_D2.5mm_P10.16mm_Horizontal"
 			(at 35.56 123.698 90)
 			(effects
@@
 			)
 		)
-		(property "Footprint" "Resistor_SMD:R_0603_1608Metric"
+		(property "Footprint" "Resistor_THT:R_Axial_DIN0207_L6.3mm_D2.5mm_P10.16mm_Horizontal"
 			(at 35.56 187.198 90)
 			(effects
@@
 		(dnp no)
 		(fields_autoplaced yes)
-		(property "Reference" "SW3"
+		(property "Reference" "SW20"
 			(at 62.23 60.96 0)
 			(effects
@@
 			(project "DYI_CDJ_v1"
 				(path "/f67f3c27-8ae6-4ed2-82a6-2d91869979e0"
-					(reference "SW3")
+					(reference "SW20")
 					(unit 1)
 				)
@@
 			)
 		)
-		(property "Footprint" "Resistor_SMD:R_0603_1608Metric"
+		(property "Footprint" "Resistor_THT:R_Axial_DIN0207_L6.3mm_D2.5mm_P10.16mm_Horizontal"
 			(at 35.56 51.308 90)
 			(effects
@@
 			)
 		)
-		(property "Footprint" "Resistor_SMD:R_0603_1608Metric"
+		(property "Footprint" "Resistor_THT:R_Axial_DIN0207_L6.3mm_D2.5mm_P10.16mm_Horizontal"
 			(at 35.56 234.188 90)
 			(effects
@@
 		(dnp no)
 		(fields_autoplaced yes)
-		(property "Reference" "SW15"
+		(property "Reference" "SW2"
 			(at 62.23 252.73 0)
 			(effects
@@
 			(project "DYI_CDJ_v1"
 				(path "/f67f3c27-8ae6-4ed2-82a6-2d91869979e0"
-					(reference "SW15")
+					(reference "SW2")
 					(unit 1)
 				)
@@
 			)
 		)
-		(property "Footprint" "Resistor_SMD:R_0603_1608Metric"
+		(property "Footprint" "Resistor_THT:R_Axial_DIN0207_L6.3mm_D2.5mm_P10.16mm_Horizontal"
 			(at 35.56 279.908 90)
 			(effects
@@
 			)
 		)
-		(property "Footprint" "Resistor_SMD:R_0603_1608Metric"
+		(property "Footprint" "Resistor_THT:R_Axial_DIN0207_L6.3mm_D2.5mm_P10.16mm_Horizontal"
 			(at 35.56 32.258 90)
 			(effects
@@
 		(dnp no)
 		(fields_autoplaced yes)
-		(property "Reference" "SW12"
+		(property "Reference" "SW15"
 			(at 62.23 210.82 0)
 			(effects
@@
 			(project "DYI_CDJ_v1"
 				(path "/f67f3c27-8ae6-4ed2-82a6-2d91869979e0"
-					(reference "SW12")
+					(reference "SW15")
 					(unit 1)
 				)
@@
 			)
 		)
-		(property "Footprint" "Resistor_SMD:R_0603_1608Metric"
+		(property "Footprint" "Resistor_THT:R_Axial_DIN0207_L6.3mm_D2.5mm_P10.16mm_Horizontal"
 			(at 35.56 262.128 90)
 			(effects
@@
 			)
 		)
-		(property "Footprint" "Resistor_SMD:R_0603_1608Metric"
+		(property "Footprint" "Resistor_THT:R_Axial_DIN0207_L6.3mm_D2.5mm_P10.16mm_Horizontal"
 			(at 35.56 204.978 90)
 			(effects
